File: tmc5160_step.brd (EAGLE design)
At the start: 160 x 100 mm, 180 parts, among them IC1 MEGA32-A, IC2 ZR78LXXG, IC4 TMC5160-TA, IC7 MAX3072EESA, IC8 MAX1776

Commit message: tmc4361 hinzugefügt
Parts:
- removed R3, R4: 2K2, rcl-2:R0603
- added C41, C42, C43, C44, C9: 470nF, rcl:C0603
- added C45, C46: 100nF, rcl-2:C0603
- added IC5: TMC4361A-LA, TMC4361A-LA:TMC_QFN40_0.5_6.0X6.0
- C21: value 100nF -> 470nF
- OK1, OK4: value HCPL2430SOIC08 -> HCPL0601
- moved C21 48.5 mm to (50.7, 76.3), flipped to the top, turned to 0 degrees
- moved H3 10.3 mm to (139.5, 94.4)
- moved H2 10.3 mm to (79.1, 94.4)
- moved OK4 0.40 mm to (67.1, 58.1), turned to 0 degrees
- moved OK1 0.28 mm to (54.3, 61.7), turned to 0 degrees
Connections:
- removed net N$36: OK1.3, R39.1
- removed net VREF: R4.2
- removed net VS: IC4.33
- new net N$12: C43.1, IC5.35
- net +3V3: now also C21.1, C41.1, C42.1, C45.1, C46.1, IC5.26, IC5.37, IC5.5, OK1.8, OK4.8
- net DGND: now also C41.2, C42.2, C43.2, C44.2, C45.2, C46.2, IC5.15, IC5.25, IC5.36, IC5.41, IC5.6, OK1.5, OK4.5
- net N$21: now also C44.1, IC5.16; no longer IC1.14, R3.1
- net N$22: now also OK1.3, R33.1; no longer C21.1, R3.2, R4.1
- net N$25: now also R39.1; no longer R33.1
- net STEP_DIR: now also OK1.6; no longer OK4.6
- net STEP_SYNC: now also OK4.6; no longer OK1.6
- net VBUS: now also C9.2, IC4.33
- net VEE: now also OK1.2, OK4.2; no longer OK1.4, OK4.4
Routing:
- net IF_PWR: track 58.5 -> 3.63 mm
- net N$21: track 33.4 -> 0.00 mm, vias 1 -> 0
- net PE: track 785.7 -> 756.6 mm
- net N$18: track 46.8 -> 19.9 mm
- net N$19: track 43.7 -> 20.8 mm
- net N$17: track 37.9 -> 16.5 mm
- net N$16: track 36.1 -> 16.8 mm
- net N$14: track 47.1 -> 34.1 mm
- net N$22: track 6.40 -> 0.00 mm
- net N$13: track 4.11 -> 0.00 mm
- net N$25: track 2.10 -> 0.00 mm
- net STEP_DIR: track 26.5 -> 24.5 mm
- net N$36: track 2.05 -> 0.00 mm
- net VREF: track 1.64 -> 0.00 mm, vias 1 -> 0
