File: tmc5160_step.sch (EAGLE design)
At the start: 180 parts, among them IC1 MEGA32-A, IC2 ZR78LXXG, IC4 TMC5160-TA, IC7 MAX3072EESA, IC8 MAX1776

Commit message: tmc4361 hinzugefügt
Parts:
- removed R3, R4: 2K2, rcl-2:R-EU_R0603
- added C41, C42, C43, C44, C9: 470nF, rcl:C-EUC0603
- added C45, C46: 100nF, rcl-2:C-EUC0603
- added IC5: TMC4361A-LA, TMC4361A-LA:TMC4361A-LA
- C21: value 100nF -> 470nF
- OK1, OK4: value HCPL2430SOIC08 -> HCPL0601; device optocoupler:HCPL2430SOIC08 -> optocoupler:HCPL0601
Connections:
- removed net N$36: OK1B.C, R39.1
- removed net VREF: R4.2
- new net N$12: C43.1, IC5.VDD1V8_2
- net +3V3: now also C21.1, C41.1, C42.1, C45.1, C46.1, IC5.VCC_1, IC5.VCC_2, IC5.VCC_3, OK1.VCC, OK4.VCC
- net DGND: now also C41.2, C42.2, C43.2, C44.2, C45.2, C46.2, IC5.GND_1, IC5.GND_2, IC5.GND_3, IC5.GND_4, IC5.GND_PAD, OK1.GND, OK4.GND
- net N$21: now also C44.1, IC5.VDD1V8_1; no longer IC1.(OC1A)PD5, R3.1
- net N$22: now also OK1.C, R33.1; no longer C21.1, R3.2, R4.1
- net N$25: now also OK4.C, R39.1; no longer OK4B.C, R33.1
- net STEP_DIR: now also OK1.VO; no longer OK4B.OUT
- net STEP_SYNC: now also OK4.VO; no longer OK1B.OUT
- net VBUS: now also C9.2, IC4.VS
- net VEE: now also OK1.A, OK4.A; no longer OK1B.A, OK4B.A
